File: robot/schematElektryczny/ledyyy.kicad_sch (KiCad schematic)
At the start: 3 parts

Commit message: ok
Parts:
- gave numbers to parts that had none: 3
Changed lines of the file:
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@@
   (symbol (lib_id "LED:WS2812B") (at 138.43 78.105 0) (unit 1)
     (in_bom yes) (on_board yes) (fields_autoplaced)
-    (property "Reference" "D?" (id 0) (at 149.86 73.7743 0))
+    (property "Reference" "D13" (id 0) (at 149.86 73.7743 0))
     (property "Value" "WS2812B" (id 1) (at 149.86 76.3143 0))
     (property "Footprint" "LED_SMD:LED_WS2812B_PLCC4_5.0x5.0mm_P3.2mm" (id 2) (at 139.7 85.725 0)
@@
   (symbol (lib_id "power:+5V") (at 85.725 93.98 180) (unit 1)
     (in_bom yes) (on_board yes) (fields_autoplaced)
-    (property "Reference" "#PWR?" (id 0) (at 85.725 90.17 0)
+    (property "Reference" "#PWR0123" (id 0) (at 85.725 90.17 0)
       (effects (font (size 1.27 1.27)) hide)
     )
@@
   (symbol (lib_id "LED:WS2812B") (at 113.03 78.105 0) (unit 1)
     (in_bom yes) (on_board yes) (fields_autoplaced)
-    (property "Reference" "D?" (id 0) (at 124.46 73.7743 0))
+    (property "Reference" "D12" (id 0) (at 124.46 73.7743 0))
     (property "Value" "WS2812B" (id 1) (at 124.46 76.3143 0))
     (property "Footprint" "LED_SMD:LED_WS2812B_PLCC4_5.0x5.0mm_P3.2mm" (id 2) (at 114.3 85.725 0)
@@
   (symbol (lib_id "power:GND") (at 85.725 60.96 180) (unit 1)
     (in_bom yes) (on_board yes) (fields_autoplaced)
-    (property "Reference" "#PWR?" (id 0) (at 85.725 54.61 0)
+    (property "Reference" "#PWR0124" (id 0) (at 85.725 54.61 0)
       (effects (font (size 1.27 1.27)) hide)
     )
@@
   (symbol (lib_id "LED:WS2812B") (at 85.725 78.105 0) (unit 1)
     (in_bom yes) (on_board yes) (fields_autoplaced)
-    (property "Reference" "D?" (id 0) (at 97.155 73.7743 0))
+    (property "Reference" "D11" (id 0) (at 97.155 73.7743 0))
     (property "Value" "WS2812B" (id 1) (at 97.155 76.3143 0))
     (property "Footprint" "LED_SMD:LED_WS2812B_PLCC4_5.0x5.0mm_P3.2mm" (id 2) (at 86.995 85.725 0)
