File: robot/schematElektryczny/motorController.kicad_sch (KiCad schematic)
At the start: 33 parts

Commit message: ok
Parts:
- removed C?: C, symbol Device:C
- removed JP? (x2): Jumper_2_Open, Jumper:SolderJumper-2_P1.3mm_Open_TrianglePad1.0x1.5mm, symbol Jumper:Jumper_2_Open
- removed Q? (x4): 2N3904, Package_TO_SOT_THT:TO-92_Inline, symbol Transistor_BJT:2N3904
- removed R? (x14): R, symbol Device:R
- added C9: C_Polarized, Capacitor_THT:CP_Radial_D10.0mm_P5.00mm, symbol Device:C_Polarized
- C2: renamed from C?; footprint (none) -> Capacitor_THT:C_Disc_D5.0mm_W2.5mm_P2.50mm
- D10, D3, D4, D5, D6, D7, D8, D9: renamed from D?; footprint (none) -> Diode_SMD:D_SOD-128
- J2, J3: renamed from J?; footprint (none) -> Connector_Hirose:Hirose_DF13C_CL535-0406-3-51_1x06-1MP_P1.25mm_Vertical
- gave numbers to parts that had none: 1
Connections:
- net 5V_IN: no longer J2.6 (Pin_6), J3.6 (Pin_6)
- net ENCO_1: now also J3.3 (Pin_3)
- net ENCO_2: now also J2.3 (Pin_3)
- net GND: now also C9.2
- net M1_1: now also J2.1 (Pin_1)
- net M2_1: now also J3.1 (Pin_1)
- net MOTOR_VOLTAGE: now also C9.1
- net PWM_M2_1: now reaches U3.10 (IN3)
- net PWM_M2_2: now reaches U3.12 (IN4)
- net PWM_M1_1: now reaches U3.5 (IN1)
- net PWM_M1_2: now reaches U3.7 (IN2)
- new net 3V3_IN: J2.6 (Pin_6), J3.6 (Pin_6)
Other:
- note removed: "5V --> 3.3V Logic"
- moved on the sheet: J2, J3
