File: robot/schematElektryczny/psu.kicad_sch (KiCad schematic)
At the start: 22 parts

Commit message: ok
Parts:
- removed C? (x4): C, symbol Device:C
- removed C? (x2): C_Polarized, symbol Device:C_Polarized
- removed D? (x2): D, symbol Device:D
- removed R? (x4): R, symbol Device:R
- removed U? (x2): AMS1117, Package_TO_SOT_SMD:SOT-223-3_TabPin2, symbol Regulator_Linear:AMS1117
- removed U?: LM7812_TO220, Package_TO_SOT_THT:TO-220-3_Vertical, symbol Regulator_Linear:LM7812_TO220
- added C1, C6: C_Polarized, Capacitor_THT:CP_Radial_D8.0mm_P5.00mm, symbol Device:C_Polarized
- added C4, C5: C, Capacitor_THT:C_Disc_D5.0mm_W2.5mm_P5.00mm, symbol Device:C
- added U2: L7805, symbol Regulator_Linear:L7805
- D1: renamed from D?; footprint (none) -> Diode_THT:D_DO-15_P10.16mm_Horizontal
- D2: renamed from D?; footprint (none) -> LED_THT:LED_D3.0mm
- F1: renamed from F?; footprint (none) -> Fuse:Fuse_1210_3225Metric_Pad1.42x2.65mm_HandSolder
- J1: renamed from J?; footprint (none) -> TerminalBlock:TerminalBlock_bornier-2_P5.08mm
- R1, R2, R5: renamed from R?; footprint (none) -> Resistor_THT:R_Axial_DIN0207_L6.3mm_D2.5mm_P10.16mm_Horizontal
Connections:
- net +12V is gone; now on net +BATT: D1.1 (K)
- net +3V3 is gone; now on net +5V: D2.2 (A)
- net +5V: now also C5.1, C6.1, U2.3 (OUT)
- net +BATT: now also C1.1, C4.1, U2.1 (IN)
- net -BATT: now also C1.2, C4.2, C5.2, C6.2, U2.2 (GND)
Other:
- note removed: "TODO: rezystory"
- moved on the sheet: D1, D2, R5
