File: robot/schematElektryczny/robot.kicad_sch (KiCad schematic)
At the start: 1 part

Commit message: ok
Parts:
- removed U?: ESP32-WROOM-32, RF_Module:ESP32-WROOM-32, symbol RF_Module:ESP32-WROOM-32
- added C3, C7: C, Capacitor_THT:C_Disc_D5.0mm_W2.5mm_P5.00mm, symbol Device:C
- added C8: C_Polarized, Capacitor_THT:CP_Radial_D10.0mm_P5.00mm, symbol Device:C_Polarized
- added U1: ESP32_NODEMCU, footprints:MODULE_ESP32_NODEMCU, symbol ESP32_NODEMCU:ESP32_NODEMCU
Connections:
- net +5V: now also C3.2, U1.J5_1 (5V)
- net GND: now also C3.1, C7.1, C8.2, U1.J4_1 (GND), U1.J4_7 (GND), U1.J5_6 (GND)
- new net +3.3V: C7.2, C8.1, U1.J5_19 (3V3)
- new net BATT_VOLTAGE_DIVIDER: U1.J5_14 (G35)
- new net ENCO_1: U1.J4_13 (G4)
- new net ENCO_2: U1.J4_2 (G23)
- new net LED_OUT: U1.J4_10 (G5)
- new net PWM_M1_1: U1.J4_3 (G22)
- new net PWM_M1_2: U1.J4_6 (G21)
- new net PWM_M2_1: U1.J4_8 (G19)
- new net PWM_M2_2: U1.J4_9 (G18)
Other:
- sheet motorController ports: added 3V3_IN, PWM_M1_1, PWM_M1_2, PWM_M2_1, PWM_M2_2; removed M1_1, M1_2, M2_1, M2_2
